File: Plaquette de montage/Plaquette de montage.kicad_pcb (KiCad board)
At the start: 2 copper layers, 40 x 69 mm, 38 parts, among them J1 Conn_01x06_Pin, J2 Conn_01x06_Pin, Q1 2N3904, Q2 2N3904, Q3 2N3904, SW1 LED_switch, U1 MCP6004

Commit message: Ajout des ground plane et des via stitching
Parts:
- added D4: LED, LED_THT:LED_D5.0mm, F.Cu at (205.7, 77.7)
- added R21: 150, Resistor_THT:R_Axial_DIN0207_L6.3mm_D2.5mm_P10.16mm_Horizontal, F.Cu at (225.0, 79.6)
- moved G*** 1.13 mm to (206.9, 66.3)
Routing:
- net Net-(D4-K): track 0.00 -> 22.7 mm
- net GND: track 122.1 -> 133.6 mm, vias 1 -> 67
- net +5V: track 118.1 -> 120.5 mm
- added copper zone on B.Cu, net GND
- added copper zone on F.Cu, net GND
Other:
- board size 40 x 69 mm -> 40.2 x 69 mm
