File: Plaquette de montage/Plaquette de montage.kicad_sch (KiCad schematic)
At the start: 37 parts, among them J1 Conn_01x06_Pin, J2 Conn_01x06_Pin, Q1 2N3904, Q2 2N3904, Q3 2N3904, SW1 LED_switch, U1 MCP6004

Commit message: Ajout des ground plane et des via stitching
Parts:
- added D4: LED, LED_THT:LED_D5.0mm, symbol Device:LED
- added R21: 150, Resistor_THT:R_Axial_DIN0207_L6.3mm_D2.5mm_P10.16mm_Horizontal, symbol Device:R_US
Connections:
- net +5V: now also D4.2 (A)
- net GND: now also R21.2
- new net: D4.1 (K), R21.1
Other:
- note added: "DEL Alimentation"
